Commit message: Added .obj mesh option in WX250S URDF/Xacro

File: interbotix_ros_xsarms/interbotix_xsarm_descriptions/urdf/wx250s.urdf.xacro (robot description, xacro)
@@ -9,4 +9,5 @@
   <xacro:arg name="external_urdf_loc" default=""/>
   <xacro:arg name="load_gazebo_configs" default="false"/>
+  <xacro:arg name="mesh_format" default="stl"/>
   <xacro:property name="urdf_loc" value="$(arg external_urdf_loc)"/>
   <xacro:property name="pi_offset" value="0.00001"/>
@@ -28,12 +29,12 @@
       <origin rpy="0 0 ${pi/2}" xyz="0 0 0"/>
       <geometry>
-        <mesh filename="package://interbotix_xsarm_descriptions/meshes/wx250s_meshes/wx250s_1_base.stl" scale="0.001 0.001 0.001"/>
-      </geometry>
-      <material name="interbotix_black"/>
-    </visual>
-    <collision>
-      <origin rpy="0 0 ${pi/2}" xyz="0 0 0"/>
-      <geometry>
-        <mesh filename="package://interbotix_xsarm_descriptions/meshes/wx250s_meshes/wx250s_1_base.stl" scale="0.001 0.001 0.001"/>
+        <mesh filename="package://interbotix_xsarm_descriptions/meshes/wx250s_meshes/wx250s_1_base.$(arg mesh_format)" scale="0.001 0.001 0.001"/>
+      </geometry>
+      <material name="interbotix_black"/>
+    </visual>
+    <collision>
+      <origin rpy="0 0 ${pi/2}" xyz="0 0 0"/>
+      <geometry>
+        <mesh filename="package://interbotix_xsarm_descriptions/meshes/wx250s_meshes/wx250s_1_base.$(arg mesh_format)" scale="0.001 0.001 0.001"/>
       </geometry>
     </collision>
@@ -65,5 +66,5 @@
       <origin rpy="0 0 ${pi/2}" xyz="0 0 -0.003"/>
       <geometry>
-        <mesh filename="package://interbotix_xsarm_descriptions/meshes/wx250s_meshes/wx250s_2_shoulder.stl" scale="0.001 0.001 0.001"/>
+        <mesh filename="package://interbotix_xsarm_descriptions/meshes/wx250s_meshes/wx250s_2_shoulder.$(arg mesh_format)" scale="0.001 0.001 0.001"/>
       </geometry>
       <material name="interbotix_black"/>
@@ -72,5 +73,5 @@
       <origin rpy="0 0 ${pi/2}" xyz="0 0 -0.003"/>
       <geometry>
-        <mesh filename="package://interbotix_xsarm_descriptions/meshes/wx250s_meshes/wx250s_2_shoulder.stl" scale="0.001 0.001 0.001"/>
+        <mesh filename="package://interbotix_xsarm_descriptions/meshes/wx250s_meshes/wx250s_2_shoulder.$(arg mesh_format)" scale="0.001 0.001 0.001"/>
       </geometry>
     </collision>
@@ -102,12 +103,12 @@
       <origin rpy="0 0 ${pi/2}" xyz="0 0 0"/>
       <geometry>
-        <mesh filename="package://interbotix_xsarm_descriptions/meshes/wx250s_meshes/wx250s_3_upper_arm.stl" scale="0.001 0.001 0.001"/>
-      </geometry>
-      <material name="interbotix_black"/>
-    </visual>
-    <collision>
-      <origin rpy="0 0 ${pi/2}" xyz="0 0 0"/>
-      <geometry>
-        <mesh filename="package://interbotix_xsarm_descriptions/meshes/wx250s_meshes/wx250s_3_upper_arm.stl" scale="0.001 0.001 0.001"/>
+        <mesh filename="package://interbotix_xsarm_descriptions/meshes/wx250s_meshes/wx250s_3_upper_arm.$(arg mesh_format)" scale="0.001 0.001 0.001"/>
+      </geometry>
+      <material name="interbotix_black"/>
+    </visual>
+    <collision>
+      <origin rpy="0 0 ${pi/2}" xyz="0 0 0"/>
+      <geometry>
+        <mesh filename="package://interbotix_xsarm_descriptions/meshes/wx250s_meshes/wx250s_3_upper_arm.$(arg mesh_format)" scale="0.001 0.001 0.001"/>
       </geometry>
     </collision>
@@ -139,5 +140,5 @@
       <origin rpy="0 0 0" xyz="0 0 0"/>
       <geometry>
-        <mesh filename="package://interbotix_xsarm_descriptions/meshes/wx250s_meshes/wx250s_4_upper_forearm.stl" scale="0.001 0.001 0.001"/>
+        <mesh filename="package://interbotix_xsarm_descriptions/meshes/wx250s_meshes/wx250s_4_upper_forearm.$(arg mesh_format)" scale="0.001 0.001 0.001"/>
       </geometry>
       <material name="interbotix_black"/>
@@ -146,5 +147,5 @@
       <origin rpy="0 0 0" xyz="0 0 0"/>
       <geometry>
-        <mesh filename="package://interbotix_xsarm_descriptions/meshes/wx250s_meshes/wx250s_4_upper_forearm.stl" scale="0.001 0.001 0.001"/>
+        <mesh filename="package://interbotix_xsarm_descriptions/meshes/wx250s_meshes/wx250s_4_upper_forearm.$(arg mesh_format)" scale="0.001 0.001 0.001"/>
       </geometry>
     </collision>
@@ -176,5 +177,5 @@
       <origin rpy="${pi} 0 0" xyz="0 0 0"/>
       <geometry>
-        <mesh filename="package://interbotix_xsarm_descriptions/meshes/wx250s_meshes/wx250s_5_lower_forearm.stl" scale="0.001 0.001 0.001"/>
+        <mesh filename="package://interbotix_xsarm_descriptions/meshes/wx250s_meshes/wx250s_5_lower_forearm.$(arg mesh_format)" scale="0.001 0.001 0.001"/>
       </geometry>
       <material name="interbotix_black"/>
@@ -183,5 +184,5 @@
       <origin rpy="${pi} 0 0" xyz="0 0 0"/>
       <geometry>
-        <mesh filename="package://interbotix_xsarm_descriptions/meshes/wx250s_meshes/wx250s_5_lower_forearm.stl" scale="0.001 0.001 0.001"/>
+        <mesh filename="package://interbotix_xsarm_descriptions/meshes/wx250s_meshes/wx250s_5_lower_forearm.$(arg mesh_format)" scale="0.001 0.001 0.001"/>
       </geometry>
     </collision>
@@ -213,12 +214,12 @@
       <origin rpy="0 0 ${pi/2}" xyz="0 0 0"/>
       <geometry>
-        <mesh filename="package://interbotix_xsarm_descriptions/meshes/wx250s_meshes/wx250s_6_wrist.stl" scale="0.001 0.001 0.001"/>
-      </geometry>
-      <material name="interbotix_black"/>
-    </visual>
-    <collision>
-      <origin rpy="0 0 ${pi/2}" xyz="0 0 0"/>
-      <geometry>
-        <mesh filename="package://interbotix_xsarm_descriptions/meshes/wx250s_meshes/wx250s_6_wrist.stl" scale="0.001 0.001 0.001"/>
+        <mesh filename="package://interbotix_xsarm_descriptions/meshes/wx250s_meshes/wx250s_6_wrist.$(arg mesh_format)" scale="0.001 0.001 0.001"/>
+      </geometry>
+      <material name="interbotix_black"/>
+    </visual>
+    <collision>
+      <origin rpy="0 0 ${pi/2}" xyz="0 0 0"/>
+      <geometry>
+        <mesh filename="package://interbotix_xsarm_descriptions/meshes/wx250s_meshes/wx250s_6_wrist.$(arg mesh_format)" scale="0.001 0.001 0.001"/>
       </geometry>
     </collision>
@@ -250,5 +251,5 @@
       <origin rpy="0 0 ${pi/2}" xyz="-0.02 0 0"/>
       <geometry>
-        <mesh filename="package://interbotix_xsarm_descriptions/meshes/wx250s_meshes/wx250s_7_gripper.stl" scale="0.001 0.001 0.001"/>
+        <mesh filename="package://interbotix_xsarm_descriptions/meshes/wx250s_meshes/wx250s_7_gripper.$(arg mesh_format)" scale="0.001 0.001 0.001"/>
       </geometry>
       <material name="interbotix_black"/>
@@ -257,5 +258,5 @@
       <origin rpy="0 0 ${pi/2}" xyz="-0.02 0 0"/>
       <geometry>
-        <mesh filename="package://interbotix_xsarm_descriptions/meshes/wx250s_meshes/wx250s_7_gripper.stl" scale="0.001 0.001 0.001"/>
+        <mesh filename="package://interbotix_xsarm_descriptions/meshes/wx250s_meshes/wx250s_7_gripper.$(arg mesh_format)" scale="0.001 0.001 0.001"/>
       </geometry>
     </collision>
@@ -299,5 +300,5 @@
       <origin rpy="0 0 ${pi/2}" xyz="-0.0685 0 0"/>
       <geometry>
-        <mesh filename="package://interbotix_xsarm_descriptions/meshes/wx250s_meshes/wx250s_8_gripper_prop.stl" scale="0.001 0.001 0.001"/>
+        <mesh filename="package://interbotix_xsarm_descriptions/meshes/wx250s_meshes/wx250s_8_gripper_prop.$(arg mesh_format)" scale="0.001 0.001 0.001"/>
       </geometry>
       <material name="interbotix_black"/>
@@ -306,5 +307,5 @@
       <origin rpy="0 0 ${pi/2}" xyz="-0.0685 0 0"/>
       <geometry>
-        <mesh filename="package://interbotix_xsarm_descriptions/meshes/wx250s_meshes/wx250s_8_gripper_prop.stl" scale="0.001 0.001 0.001"/>
+        <mesh filename="package://interbotix_xsarm_descriptions/meshes/wx250s_meshes/wx250s_8_gripper_prop.$(arg mesh_format)" scale="0.001 0.001 0.001"/>
       </geometry>
     </collision>
@@ -327,5 +328,5 @@
         <origin rpy="0 0 0" xyz="0 0 0"/>
         <geometry>
-          <mesh filename="package://interbotix_xsarm_descriptions/meshes/wx250s_meshes/wx250s_11_ar_tag.stl" scale="0.001 0.001 0.001"/>
+          <mesh filename="package://interbotix_xsarm_descriptions/meshes/wx250s_meshes/wx250s_11_ar_tag.$(arg mesh_format)" scale="0.001 0.001 0.001"/>
         </geometry>
         <material name="interbotix_black"/>
@@ -334,5 +335,5 @@
         <origin rpy="0 0 0" xyz="0 0 0"/>
         <geometry>
-          <mesh filename="package://interbotix_xsarm_descriptions/meshes/wx250s_meshes/wx250s_11_ar_tag.stl" scale="0.001 0.001 0.001"/>
+          <mesh filename="package://interbotix_xsarm_descriptions/meshes/wx250s_meshes/wx250s_11_ar_tag.$(arg mesh_format)" scale="0.001 0.001 0.001"/>
         </geometry>
       </collision>
@@ -356,5 +357,5 @@
         <origin rpy="0 0 ${pi/2}" xyz="-0.063 0 0"/>
         <geometry>
-          <mesh filename="package://interbotix_xsarm_descriptions/meshes/wx250s_meshes/wx250s_9_gripper_bar.stl" scale="0.001 0.001 0.001"/>
+          <mesh filename="package://interbotix_xsarm_descriptions/meshes/wx250s_meshes/wx250s_9_gripper_bar.$(arg mesh_format)" scale="0.001 0.001 0.001"/>
         </geometry>
         <material name="interbotix_black"/>
@@ -363,5 +364,5 @@
         <origin rpy="0 0 ${pi/2}" xyz="-0.063 0 0"/>
         <geometry>
-          <mesh filename="package://interbotix_xsarm_descriptions/meshes/wx250s_meshes/wx250s_9_gripper_bar.stl" scale="0.001 0.001 0.001"/>
+          <mesh filename="package://interbotix_xsarm_descriptions/meshes/wx250s_meshes/wx250s_9_gripper_bar.$(arg mesh_format)" scale="0.001 0.001 0.001"/>
         </geometry>
       </collision>
@@ -407,5 +408,5 @@
           <origin rpy="${pi} ${pi} 0" xyz="0 0.005 0"/>
           <geometry>
-            <mesh filename="package://interbotix_xsarm_descriptions/meshes/wx250s_meshes/wx250s_10_gripper_finger.stl" scale="0.001 0.001 0.001"/>
+            <mesh filename="package://interbotix_xsarm_descriptions/meshes/wx250s_meshes/wx250s_10_gripper_finger.$(arg mesh_format)" scale="0.001 0.001 0.001"/>
           </geometry>
           <material name="interbotix_black"/>
@@ -414,5 +415,5 @@
           <origin rpy="${pi} ${pi} 0" xyz="0 0.005 0"/>
           <geometry>
-            <mesh filename="package://interbotix_xsarm_descriptions/meshes/wx250s_meshes/wx250s_10_gripper_finger.stl" scale="0.001 0.001 0.001"/>
+            <mesh filename="package://interbotix_xsarm_descriptions/meshes/wx250s_meshes/wx250s_10_gripper_finger.$(arg mesh_format)" scale="0.001 0.001 0.001"/>
           </geometry>
         </collision>
@@ -447,5 +448,5 @@
           <origin rpy="0 ${pi} 0" xyz="0 -0.005 0"/>
           <geometry>
-            <mesh filename="package://interbotix_xsarm_descriptions/meshes/wx250s_meshes/wx250s_10_gripper_finger.stl" scale="0.001 0.001 0.001"/>
+            <mesh filename="package://interbotix_xsarm_descriptions/meshes/wx250s_meshes/wx250s_10_gripper_finger.$(arg mesh_format)" scale="0.001 0.001 0.001"/>
           </geometry>
           <material name="interbotix_black"/>
@@ -454,5 +455,5 @@
           <origin rpy="0 ${pi} 0" xyz="0 -0.005 0"/>
           <geometry>
-            <mesh filename="package://interbotix_xsarm_descriptions/meshes/wx250s_meshes/wx250s_10_gripper_finger.stl" scale="0.001 0.001 0.001"/>
+            <mesh filename="package://interbotix_xsarm_descriptions/meshes/wx250s_meshes/wx250s_10_gripper_finger.$(arg mesh_format)" scale="0.001 0.001 0.001"/>
           </geometry>
         </collision>
